Commit message: Crane visualization

File: crane_description/urdf/crane.xacro (robot description, xacro)
@@ -2,5 +2,5 @@
 <robot xmlns:xacro="http://www.ros.org/wiki/xacro">
   <xacro:macro name="crane">
-    <link name="base_link">
+    <link name="KingBot">
       <inertial>
         <origin xyz="0 0 0" rpy="0 0 0"/>
@@ -9,10 +9,30 @@
       </inertial>
       <visual>
-        <origin xyz="0 0 0" rpy="0 0 0"/>
+        <origin xyz="0 0 0" rpy="${-pi/2} 0 0"/>
         <geometry>
-          <mesh filename="package://crane_description/meshes/visual/Cylind01.stl" scale="0.001 0.001 0.001" />
+          <mesh filename="package://crane_description/meshes/visual/KingBot.stl" scale="0.001 0.001 0.001" />
         </geometry>
       </visual>
     </link>
+    <link name="King">
+      <inertial>
+        <origin xyz="0 0 0" rpy="0 0 0"/>
+        <mass value="2"/>
+        <inertia ixx="0.01" ixy="0" ixz="0" iyy="0.01" iyz="0" izz="0.01" />
+      </inertial>
+      <visual>
+        <origin xyz="0 0 0" rpy="${-pi/2} 0 0"/>
+        <geometry>
+          <mesh filename="package://crane_description/meshes/visual/King.stl" scale="0.001 0.001 0.001" />
+        </geometry>
+      </visual>
+    </link>
+    <joint name="joint_a1" type="revolute">
+      <origin xyz="0 0 0" rpy="0 0 0"/>
+      <parent link="KingBot"/>
+      <child link="King"/>
+      <axis xyz="0 0 1"/>
+      <limit effort="0" lower="${radians(-185)}" upper="${radians(185)}" velocity="${radians(156)}"/>
+    </joint>
   </xacro:macro>
 </robot>

Commit message: Scaling

File: crane_description/urdf/crane.xacro (robot description, xacro)
@@ -9,7 +9,7 @@
       </inertial>
       <visual>
-        <origin xyz="0 0 0" rpy="${-pi/2} 0 0"/>
+        <origin xyz="0 0 0" rpy="0 0 0"/>
         <geometry>
-          <mesh filename="package://crane_description/meshes/visual/KingBot.stl" scale="0.001 0.001 0.001" />
+          <mesh filename="package://crane_description/meshes/visual/KingBot.stl" />
         </geometry>
       </visual>
@@ -22,5 +22,5 @@
       </inertial>
       <visual>
-        <origin xyz="0 0 0" rpy="${-pi/2} 0 0"/>
+        <origin xyz="0 0 3" rpy="0 0 0"/>
         <geometry>
           <mesh filename="package://crane_description/meshes/visual/King.stl" scale="0.001 0.001 0.001" />
@@ -28,6 +28,6 @@
       </visual>
     </link>
-    <joint name="joint_a1" type="revolute">
-      <origin xyz="0 0 0" rpy="0 0 0"/>
+    <joint name="joint_1" type="revolute">
+      <origin xyz="0 0 0.623" rpy="0 0 0"/>
       <parent link="KingBot"/>
       <child link="King"/>

Commit message: Two links done

File: crane_description/urdf/crane.xacro (robot description, xacro)
@@ -2,4 +2,7 @@
 <robot xmlns:xacro="http://www.ros.org/wiki/xacro">
   <xacro:macro name="crane">
+    <material name="white">
+      <color rgba="1 1 1 1"/>
+    </material>
     <link name="KingBot">
       <inertial>
@@ -13,21 +16,18 @@
           <mesh filename="package://crane_description/meshes/visual/KingBot.stl" />
         </geometry>
+        <material name="white"/>
       </visual>
     </link>
     <link name="King">
-      <inertial>
+      <visual>
         <origin xyz="0 0 0" rpy="0 0 0"/>
-        <mass value="2"/>
-        <inertia ixx="0.01" ixy="0" ixz="0" iyy="0.01" iyz="0" izz="0.01" />
-      </inertial>
-      <visual>
-        <origin xyz="0 0 3" rpy="0 0 0"/>
         <geometry>
-          <mesh filename="package://crane_description/meshes/visual/King.stl" scale="0.001 0.001 0.001" />
+          <mesh filename="package://crane_description/meshes/visual/King.stl" />
         </geometry>
+        <material name="white"/>
       </visual>
     </link>
     <joint name="joint_1" type="revolute">
-      <origin xyz="0 0 0.623" rpy="0 0 0"/>
+      <origin xyz="0 0 0.628" rpy="0 0 0"/>
       <parent link="KingBot"/>
       <child link="King"/>

Commit message: Main structure done. Working on cylinder 1

File: crane_description/urdf/crane.xacro (robot description, xacro)
@@ -28,4 +28,40 @@
       </visual>
     </link>
+    <link name="Boom1">
+      <visual>
+        <origin xyz="0 0 0" rpy="0 0 0"/>
+        <geometry>
+          <mesh filename="package://crane_description/meshes/visual/Boom1.stl" />
+        </geometry>
+        <material name="white"/>
+      </visual>
+    </link>
+    <link name="Boom2">
+      <visual>
+        <origin xyz="0 0 0" rpy="0 0 0"/>
+        <geometry>
+          <mesh filename="package://crane_description/meshes/visual/Boom2.stl" />
+        </geometry>
+        <material name="white"/>
+      </visual>
+    </link>
+    <link name="Cyl1">
+      <visual>
+        <origin xyz="0 0 0" rpy="0 0 0"/>
+        <geometry>
+          <mesh filename="package://crane_description/meshes/visual/Cyl1.stl" />
+        </geometry>
+        <material name="white"/>
+      </visual>
+    </link>
+    <link name="Piston1">
+      <visual>
+        <origin xyz="0 0 0" rpy="0 0 0"/>
+        <geometry>
+          <mesh filename="package://crane_description/meshes/visual/Piston1.stl" />
+        </geometry>
+        <material name="white"/>
+      </visual>
+    </link>
     <joint name="joint_1" type="revolute">
       <origin xyz="0 0 0.628" rpy="0 0 0"/>
@@ -35,4 +71,28 @@
       <limit effort="0" lower="${radians(-185)}" upper="${radians(185)}" velocity="${radians(156)}"/>
     </joint>
+    <joint name="joint_2" type="revolute">
+      <origin xyz="0 0 0.706" rpy="0 0 0"/>
+      <parent link="King"/>
+      <child link="Boom1"/>
+      <axis xyz="0 1 0"/>
+      <limit effort="0" lower="${radians(-90)}" upper="${0}" velocity="${radians(156)}"/>
+    </joint>
+    <joint name="joint_3" type="revolute">
+      <origin xyz="1.468171 0 0.308337" rpy="0 0 0"/>
+      <parent link="Boom1"/>
+      <child link="Boom2"/>
+      <axis xyz="0 1 0"/>
+      <limit effort="0" lower="${radians(-90)}" upper="${0}" velocity="${radians(156)}"/>
+    </joint>
+    <joint name="cyl1_joint" type="fixed">
+      <origin xyz="0.154236 0 0.116" rpy="0 0 0"/>
+      <parent link="King"/>
+      <child link="Cyl1"/>
+    </joint>
+    <joint name="cyl1_pistion1_joint" type="fixed">
+      <origin xyz="0 0 0" rpy="0 0 0"/>
+      <parent link="King"/>
+      <child link="Piston1"/>
+    </joint>
   </xacro:macro>
 </robot>

Commit message: Main structure finished.

File: crane_description/urdf/crane.xacro (robot description, xacro)
@@ -55,4 +55,13 @@
       </visual>
     </link>
+    <link name="Cyl2">
+      <visual>
+        <origin xyz="0 0 0" rpy="0 0 0"/>
+        <geometry>
+          <mesh filename="package://crane_description/meshes/visual/Cyl2.stl" />
+        </geometry>
+        <material name="white"/>
+      </visual>
+    </link>
     <link name="Piston1">
       <visual>
@@ -60,4 +69,13 @@
         <geometry>
           <mesh filename="package://crane_description/meshes/visual/Piston1.stl" />
+        </geometry>
+        <material name="white"/>
+      </visual>
+    </link>
+    <link name="Piston2">
+      <visual>
+        <origin xyz="0 0 0" rpy="0 0 0"/>
+        <geometry>
+          <mesh filename="package://crane_description/meshes/visual/Piston2.stl" />
         </geometry>
         <material name="white"/>
@@ -86,12 +104,26 @@
     </joint>
     <joint name="cyl1_joint" type="fixed">
-      <origin xyz="0.154236 0 0.116" rpy="0 0 0"/>
+      <origin xyz="0.154236 0 0.156" rpy="0 ${radians(-49.90)} 0"/>
       <parent link="King"/>
       <child link="Cyl1"/>
     </joint>
-    <joint name="cyl1_pistion1_joint" type="fixed">
+    <joint name="cyl1_pistion1_joint" type="prismatic">
       <origin xyz="0 0 0" rpy="0 0 0"/>
-      <parent link="King"/>
+      <parent link="Cyl1"/>
       <child link="Piston1"/>
+      <axis xyz="1 0 0"/>
+      <limit effort="0" lower="0" upper="0.1" velocity="${radians(156)}"/>
+    </joint>
+    <joint name="cyl2_joint" type="fixed">
+      <origin xyz="0.767068 0 0.002395" rpy="0 ${radians(-12.49)} 0"/>
+      <parent link="Boom1"/>
+      <child link="Cyl2"/>
+    </joint>
+    <joint name="cyl2_pistion2_joint" type="prismatic">
+      <origin xyz="0 0 0" rpy="0 0 0"/>
+      <parent link="Cyl2"/>
+      <child link="Piston2"/>
+      <axis xyz="1 0 0"/>
+      <limit effort="0" lower="0" upper="0.1" velocity="${radians(156)}"/>
     </joint>
   </xacro:macro>

Commit message: started on mimic joint

File: crane_description/urdf/crane.xacro (robot description, xacro)
@@ -89,11 +89,4 @@
       <limit effort="0" lower="${radians(-185)}" upper="${radians(185)}" velocity="${radians(156)}"/>
     </joint>
-    <joint name="joint_2" type="revolute">
-      <origin xyz="0 0 0.706" rpy="0 0 0"/>
-      <parent link="King"/>
-      <child link="Boom1"/>
-      <axis xyz="0 1 0"/>
-      <limit effort="0" lower="${radians(-90)}" upper="${0}" velocity="${radians(156)}"/>
-    </joint>
     <joint name="joint_3" type="revolute">
       <origin xyz="1.468171 0 0.308337" rpy="0 0 0"/>
@@ -108,5 +101,5 @@
       <child link="Cyl1"/>
     </joint>
-    <joint name="cyl1_pistion1_joint" type="prismatic">
+    <joint name="cyl1_piston1_joint" type="prismatic">
       <origin xyz="0 0 0" rpy="0 0 0"/>
       <parent link="Cyl1"/>
@@ -115,4 +108,12 @@
       <limit effort="0" lower="0" upper="0.1" velocity="${radians(156)}"/>
     </joint>
+    <joint name="joint_2" type="revolute">
+      <origin xyz="0 0 0.706" rpy="0 0 0"/>
+      <parent link="King"/>
+      <child link="Boom1"/>
+      <axis xyz="0 1 0"/>
+      <limit effort="0" lower="${radians(-90)}" upper="${0}" velocity="${radians(156)}"/>
+      <mimic joint="cyl1_piston1_joint" offset="0"/>
+    </joint>
     <joint name="cyl2_joint" type="fixed">
       <origin xyz="0.767068 0 0.002395" rpy="0 ${radians(-12.49)} 0"/>
@@ -120,5 +121,5 @@
       <child link="Cyl2"/>
     </joint>
-    <joint name="cyl2_pistion2_joint" type="prismatic">
+    <joint name="cyl2_piston2_joint" type="prismatic">
       <origin xyz="0 0 0" rpy="0 0 0"/>
       <parent link="Cyl2"/>

Commit message: Removed unused files

File: crane_description/urdf/crane.xacro (robot description, xacro)
@@ -96,9 +96,4 @@
       <limit effort="0" lower="${radians(-90)}" upper="${0}" velocity="${radians(156)}"/>
     </joint>
-    <joint name="cyl1_joint" type="fixed">
-      <origin xyz="0.154236 0 0.156" rpy="0 ${radians(-49.90)} 0"/>
-      <parent link="King"/>
-      <child link="Cyl1"/>
-    </joint>
     <joint name="cyl1_piston1_joint" type="prismatic">
       <origin xyz="0 0 0" rpy="0 0 0"/>
@@ -108,4 +103,6 @@
       <limit effort="0" lower="0" upper="0.1" velocity="${radians(156)}"/>
     </joint>
+    <xacro:property name="a1" value="0.6141172" />
+    <xacro:property name="b1" value="0.5712169" />
     <joint name="joint_2" type="revolute">
       <origin xyz="0 0 0.706" rpy="0 0 0"/>
@@ -114,5 +111,13 @@
       <axis xyz="0 1 0"/>
       <limit effort="0" lower="${radians(-90)}" upper="${0}" velocity="${radians(156)}"/>
-      <mimic joint="cyl1_piston1_joint" offset="0"/>
+      <mimic joint="cyl1_piston1_joint" multiplier="-1" offset="0"/>
+    </joint>
+    <joint name="cyl1_joint" type="revolute">
+      <origin xyz="0.154236 0 0.156" rpy="0 ${radians(-49.90)} 0"/>
+      <parent link="King"/>
+      <child link="Cyl1"/>
+      <axis xyz="0 1 0"/>
+      <limit effort="0" lower="${radians(-90)}" upper="${0}" velocity="${radians(156)}"/>
+      <mimic joint="joint_2" multiplier="1" offset="0"/>
     </joint>
     <joint name="cyl2_joint" type="fixed">

Commit message: First linkage works

File: crane_description/urdf/crane.xacro (robot description, xacro)
@@ -89,5 +89,33 @@
       <limit effort="0" lower="${radians(-185)}" upper="${radians(185)}" velocity="${radians(156)}"/>
     </joint>
-    <joint name="joint_3" type="revolute">
+    <joint name="joint_2" type="prismatic">
+      <origin xyz="0 0 0" rpy="0 0 0"/>
+      <parent link="Cyl1"/>
+      <child link="Piston1"/>
+      <axis xyz="1 0 0"/>
+      <limit effort="0" lower="0" upper="0.1" velocity="${radians(156)}"/>
+    </joint>
+    <joint name="alpha_2" type="revolute">
+      <origin xyz="0 0 0.706" rpy="0 0 0"/>
+      <parent link="King"/>
+      <child link="Boom1"/>
+      <axis xyz="0 -1 0"/>
+      <limit effort="0" lower="${radians(-90)}" upper="${0}" velocity="${radians(156)}"/>
+    </joint>
+    <joint name="beta_2" type="revolute">
+      <origin xyz="0.154236 0 0.156" rpy="0 0 0"/>
+      <parent link="King"/>
+      <child link="Cyl1"/>
+      <axis xyz="0 -1 0"/>
+      <limit effort="0" lower="${radians(-90)}" upper="${0}" velocity="${radians(156)}"/>
+    </joint>
+    <joint name="joint_3" type="prismatic">
+      <origin xyz="0 0 0" rpy="0 0 0"/>
+      <parent link="Cyl2"/>
+      <child link="Piston2"/>
+      <axis xyz="1 0 0"/>
+      <limit effort="0" lower="0" upper="0.1" velocity="${radians(156)}"/>
+    </joint>
+    <joint name="alpha_3" type="revolute">
       <origin xyz="1.468171 0 0.308337" rpy="0 0 0"/>
       <parent link="Boom1"/>
@@ -96,40 +124,10 @@
       <limit effort="0" lower="${radians(-90)}" upper="${0}" velocity="${radians(156)}"/>
     </joint>
-    <joint name="cyl1_piston1_joint" type="prismatic">
-      <origin xyz="0 0 0" rpy="0 0 0"/>
-      <parent link="Cyl1"/>
-      <child link="Piston1"/>
-      <axis xyz="1 0 0"/>
-      <limit effort="0" lower="0" upper="0.1" velocity="${radians(156)}"/>
-    </joint>
-    <xacro:property name="a1" value="0.6141172" />
-    <xacro:property name="b1" value="0.5712169" />
-    <joint name="joint_2" type="revolute">
-      <origin xyz="0 0 0.706" rpy="0 0 0"/>
-      <parent link="King"/>
-      <child link="Boom1"/>
-      <axis xyz="0 1 0"/>
-      <limit effort="0" lower="${radians(-90)}" upper="${0}" velocity="${radians(156)}"/>
-      <mimic joint="cyl1_piston1_joint" multiplier="-1" offset="0"/>
-    </joint>
-    <joint name="cyl1_joint" type="revolute">
-      <origin xyz="0.154236 0 0.156" rpy="0 ${radians(-49.90)} 0"/>
-      <parent link="King"/>
-      <child link="Cyl1"/>
-      <axis xyz="0 1 0"/>
-      <limit effort="0" lower="${radians(-90)}" upper="${0}" velocity="${radians(156)}"/>
-      <mimic joint="joint_2" multiplier="1" offset="0"/>
-    </joint>
-    <joint name="cyl2_joint" type="fixed">
+    <joint name="beta_3" type="revolute">
       <origin xyz="0.767068 0 0.002395" rpy="0 ${radians(-12.49)} 0"/>
       <parent link="Boom1"/>
       <child link="Cyl2"/>
-    </joint>
-    <joint name="cyl2_piston2_joint" type="prismatic">
-      <origin xyz="0 0 0" rpy="0 0 0"/>
-      <parent link="Cyl2"/>
-      <child link="Piston2"/>
-      <axis xyz="1 0 0"/>
-      <limit effort="0" lower="0" upper="0.1" velocity="${radians(156)}"/>
+      <axis xyz="0 1 0"/>
+      <limit effort="0" lower="${radians(-90)}" upper="${0}" velocity="${radians(156)}"/>
     </joint>
   </xacro:macro>

Commit message: Working on boom2

File: crane_description/urdf/crane.xacro (robot description, xacro)
@@ -121,12 +121,12 @@
       <parent link="Boom1"/>
       <child link="Boom2"/>
-      <axis xyz="0 1 0"/>
+      <axis xyz="0 -1 0"/>
       <limit effort="0" lower="${radians(-90)}" upper="${0}" velocity="${radians(156)}"/>
     </joint>
     <joint name="beta_3" type="revolute">
-      <origin xyz="0.767068 0 0.002395" rpy="0 ${radians(-12.49)} 0"/>
+      <origin xyz="0.767068 0 0.002395" rpy="0 0 0"/>
       <parent link="Boom1"/>
       <child link="Cyl2"/>
-      <axis xyz="0 1 0"/>
+      <axis xyz="0 -1 0"/>
       <limit effort="0" lower="${radians(-90)}" upper="${0}" velocity="${radians(156)}"/>
     </joint>

Commit message: Kinematics working

File: crane_description/urdf/crane.xacro (robot description, xacro)
@@ -4,4 +4,10 @@
     <material name="white">
       <color rgba="1 1 1 1"/>
+    </material>
+    <material name="gray">
+      <color rgba="0.5 0.5 0.5 1"/>
+    </material>
+    <material name="lessgray">
+      <color rgba="0.75 0.75 0.75 1"/>
     </material>
     <link name="KingBot">
@@ -16,5 +22,5 @@
           <mesh filename="package://crane_description/meshes/visual/KingBot.stl" />
         </geometry>
-        <material name="white"/>
+        <material name="gray"/>
       </visual>
     </link>
@@ -52,5 +58,5 @@
           <mesh filename="package://crane_description/meshes/visual/Cyl1.stl" />
         </geometry>
-        <material name="white"/>
+        <material name="gray"/>
       </visual>
     </link>
@@ -61,5 +67,5 @@
           <mesh filename="package://crane_description/meshes/visual/Cyl2.stl" />
         </geometry>
-        <material name="white"/>
+        <material name="gray"/>
       </visual>
     </link>
@@ -70,5 +76,5 @@
           <mesh filename="package://crane_description/meshes/visual/Piston1.stl" />
         </geometry>
-        <material name="white"/>
+        <material name="lessgray"/>
       </visual>
     </link>
@@ -79,5 +85,5 @@
           <mesh filename="package://crane_description/meshes/visual/Piston2.stl" />
         </geometry>
-        <material name="white"/>
+        <material name="lessgray"/>
       </visual>
     </link>

Commit message: Added crane controller skeleton

File: crane_description/urdf/crane.xacro (robot description, xacro)
@@ -88,4 +88,6 @@
       </visual>
     </link>
+    <link name="tip">
+    </link>
     <joint name="joint_1" type="revolute">
       <origin xyz="0 0 0.628" rpy="0 0 0"/>
@@ -137,4 +139,9 @@
       <limit effort="0" lower="${radians(-90)}" upper="${0}" velocity="${radians(156)}"/>
     </joint>
+    <joint name="boom2_tip" type="fixed">
+      <origin xyz="0.719737 0 -0.907615" rpy="0 0 0"/>
+      <parent link="Boom2"/>
+      <child link="tip"/>
+    </joint>
   </xacro:macro>
 </robot>

Commit message: Crane simulator

File: crane_description/urdf/crane.xacro (robot description, xacro)
@@ -52,5 +52,5 @@
       </visual>
     </link>
-    <link name="Cyl1">
+    <!-- <link name="Cyl1">
       <visual>
         <origin xyz="0 0 0" rpy="0 0 0"/>
@@ -87,5 +87,5 @@
         <material name="lessgray"/>
       </visual>
-    </link>
+    </link> -->
     <link name="tip">
     </link>
@@ -97,5 +97,5 @@
       <limit effort="0" lower="${radians(-185)}" upper="${radians(185)}" velocity="${radians(156)}"/>
     </joint>
-    <joint name="joint_2" type="prismatic">
+    <!-- <joint name="joint_2" type="prismatic">
       <origin xyz="0 0 0" rpy="0 0 0"/>
       <parent link="Cyl1"/>
@@ -103,5 +103,5 @@
       <axis xyz="1 0 0"/>
       <limit effort="0" lower="0" upper="0.1" velocity="${radians(156)}"/>
-    </joint>
+    </joint> -->
     <joint name="alpha_2" type="revolute">
       <origin xyz="0 0 0.706" rpy="0 0 0"/>
@@ -111,5 +111,5 @@
       <limit effort="0" lower="${radians(-90)}" upper="${0}" velocity="${radians(156)}"/>
     </joint>
-    <joint name="beta_2" type="revolute">
+    <!-- <joint name="beta_2" type="revolute">
       <origin xyz="0.154236 0 0.156" rpy="0 0 0"/>
       <parent link="King"/>
@@ -124,5 +124,5 @@
       <axis xyz="1 0 0"/>
       <limit effort="0" lower="0" upper="0.1" velocity="${radians(156)}"/>
-    </joint>
+    </joint> -->
     <joint name="alpha_3" type="revolute">
       <origin xyz="1.468171 0 0.308337" rpy="0 0 0"/>
@@ -132,5 +132,5 @@
       <limit effort="0" lower="${radians(-90)}" upper="${0}" velocity="${radians(156)}"/>
     </joint>
-    <joint name="beta_3" type="revolute">
+    <!-- <joint name="beta_3" type="revolute">
       <origin xyz="0.767068 0 0.002395" rpy="0 0 0"/>
       <parent link="Boom1"/>
@@ -138,5 +138,5 @@
       <axis xyz="0 -1 0"/>
       <limit effort="0" lower="${radians(-90)}" upper="${0}" velocity="${radians(156)}"/>
-    </joint>
+    </joint> -->
     <joint name="boom2_tip" type="fixed">
       <origin xyz="0.719737 0 -0.907615" rpy="0 0 0"/>

Commit message: Updated meshes to align with kinematics

File: crane_description/urdf/crane.xacro (robot description, xacro)
@@ -126,5 +126,5 @@
     </joint> -->
     <joint name="alpha_3" type="revolute">
-      <origin xyz="1.468171 0 0.308337" rpy="0 0 0"/>
+      <origin xyz="1.500199 0 0" rpy="0 0 0"/>
       <parent link="Boom1"/>
       <child link="Boom2"/>

Commit message: Updated crane with new link names

File: crane_description/urdf/crane.xacro (robot description, xacro)
@@ -11,5 +11,10 @@
       <color rgba="0.75 0.75 0.75 1"/>
     </material>
-    <link name="KingBot">
+    <link name="base_link"/>
+    <joint name="fixed" type="fixed">
+      <parent link="base_link"/>
+      <child link="link1"/>
+    </joint>
+    <link name="link1">
       <inertial>
         <origin xyz="0 0 0" rpy="0 0 0"/>
@@ -25,5 +30,5 @@
       </visual>
     </link>
-    <link name="King">
+    <link name="link2">
       <visual>
         <origin xyz="0 0 0" rpy="0 0 0"/>
@@ -34,5 +39,5 @@
       </visual>
     </link>
-    <link name="Boom1">
+    <link name="link3">
       <visual>
         <origin xyz="0 0 0" rpy="0 0 0"/>
@@ -43,5 +48,5 @@
       </visual>
     </link>
-    <link name="Boom2">
+    <link name="link4">
       <visual>
         <origin xyz="0 0 0" rpy="0 0 0"/>
@@ -88,10 +93,9 @@
       </visual>
     </link> -->
-    <link name="tip">
-    </link>
-    <joint name="joint_1" type="revolute">
+    <link name="tip"/>
+    <joint name="joint1" type="revolute">
       <origin xyz="0 0 0.628" rpy="0 0 0"/>
-      <parent link="KingBot"/>
-      <child link="King"/>
+      <parent link="link1"/>
+      <child link="link2"/>
       <axis xyz="0 0 1"/>
       <limit effort="0" lower="${radians(-185)}" upper="${radians(185)}" velocity="${radians(156)}"/>
@@ -104,8 +108,8 @@
       <limit effort="0" lower="0" upper="0.1" velocity="${radians(156)}"/>
     </joint> -->
-    <joint name="alpha_2" type="revolute">
+    <joint name="joint2" type="revolute">
       <origin xyz="0 0 0.706" rpy="0 0 0"/>
-      <parent link="King"/>
-      <child link="Boom1"/>
+      <parent link="link2"/>
+      <child link="link3"/>
       <axis xyz="0 -1 0"/>
       <limit effort="0" lower="${radians(-90)}" upper="${0}" velocity="${radians(156)}"/>
@@ -125,8 +129,8 @@
       <limit effort="0" lower="0" upper="0.1" velocity="${radians(156)}"/>
     </joint> -->
-    <joint name="alpha_3" type="revolute">
+    <joint name="joint3" type="revolute">
       <origin xyz="1.500199 0 0" rpy="0 0 0"/>
-      <parent link="Boom1"/>
-      <child link="Boom2"/>
+      <parent link="link3"/>
+      <child link="link4"/>
       <axis xyz="0 -1 0"/>
       <limit effort="0" lower="${radians(-90)}" upper="${0}" velocity="${radians(156)}"/>
@@ -139,7 +143,7 @@
       <limit effort="0" lower="${radians(-90)}" upper="${0}" velocity="${radians(156)}"/>
     </joint> -->
-    <joint name="boom2_tip" type="fixed">
-      <origin xyz="0.719737 0 -0.907615" rpy="0 0 0"/>
-      <parent link="Boom2"/>
+    <joint name="tip_joint" type="fixed">
+      <origin xyz="0.963823 0 -0.642519" rpy="0 0 0"/>
+      <parent link="link4"/>
       <child link="tip"/>
     </joint>
