Commit message: Renamed links and joints

File: crane_description/urdf/crane.xacro (robot description, xacro)
@@ -57,5 +57,5 @@
       </visual>
     </link>
-    <!-- <link name="Cyl1">
+    <link name="cylinder1">
       <visual>
         <origin xyz="0 0 0" rpy="0 0 0"/>
@@ -66,5 +66,14 @@
       </visual>
     </link>
-    <link name="Cyl2">
+    <link name="piston1">
+      <visual>
+        <origin xyz="0 0 0" rpy="0 0 0"/>
+        <geometry>
+          <mesh filename="package://crane_description/meshes/visual/Piston1.stl" />
+        </geometry>
+        <material name="lessgray"/>
+      </visual>
+    </link>
+    <link name="cylinder2">
       <visual>
         <origin xyz="0 0 0" rpy="0 0 0"/>
@@ -75,14 +84,5 @@
       </visual>
     </link>
-    <link name="Piston1">
-      <visual>
-        <origin xyz="0 0 0" rpy="0 0 0"/>
-        <geometry>
-          <mesh filename="package://crane_description/meshes/visual/Piston1.stl" />
-        </geometry>
-        <material name="lessgray"/>
-      </visual>
-    </link>
-    <link name="Piston2">
+    <link name="piston2">
       <visual>
         <origin xyz="0 0 0" rpy="0 0 0"/>
@@ -92,5 +92,5 @@
         <material name="lessgray"/>
       </visual>
-    </link> -->
+    </link>
     <link name="tip"/>
     <joint name="joint1" type="revolute">
@@ -101,11 +101,11 @@
       <limit effort="0" lower="${radians(-185)}" upper="${radians(185)}" velocity="${radians(156)}"/>
     </joint>
-    <!-- <joint name="joint_2" type="prismatic">
+    <joint name="actuator_joint2" type="prismatic">
       <origin xyz="0 0 0" rpy="0 0 0"/>
-      <parent link="Cyl1"/>
-      <child link="Piston1"/>
+      <parent link="cylinder1"/>
+      <child link="piston1"/>
       <axis xyz="1 0 0"/>
       <limit effort="0" lower="0" upper="0.1" velocity="${radians(156)}"/>
-    </joint> -->
+    </joint>
     <joint name="joint2" type="revolute">
       <origin xyz="0 0 0.706" rpy="0 0 0"/>
@@ -115,18 +115,18 @@
       <limit effort="0" lower="${radians(-90)}" upper="${0}" velocity="${radians(156)}"/>
     </joint>
-    <!-- <joint name="beta_2" type="revolute">
+    <joint name="link2_cylinder1_joint" type="revolute">
       <origin xyz="0.154236 0 0.156" rpy="0 0 0"/>
-      <parent link="King"/>
-      <child link="Cyl1"/>
+      <parent link="link2"/>
+      <child link="cylinder1"/>
       <axis xyz="0 -1 0"/>
       <limit effort="0" lower="${radians(-90)}" upper="${0}" velocity="${radians(156)}"/>
     </joint>
-    <joint name="joint_3" type="prismatic">
+    <joint name="actuator_joint3" type="prismatic">
       <origin xyz="0 0 0" rpy="0 0 0"/>
-      <parent link="Cyl2"/>
-      <child link="Piston2"/>
+      <parent link="cylinder2"/>
+      <child link="piston2"/>
       <axis xyz="1 0 0"/>
       <limit effort="0" lower="0" upper="0.1" velocity="${radians(156)}"/>
-    </joint> -->
+    </joint>
     <joint name="joint3" type="revolute">
       <origin xyz="1.500199 0 0" rpy="0 0 0"/>
@@ -136,11 +136,11 @@
       <limit effort="0" lower="${radians(-90)}" upper="${0}" velocity="${radians(156)}"/>
     </joint>
-    <!-- <joint name="beta_3" type="revolute">
+    <joint name="link3_cylinder2_joint" type="revolute">
       <origin xyz="0.767068 0 0.002395" rpy="0 0 0"/>
-      <parent link="Boom1"/>
-      <child link="Cyl2"/>
+      <parent link="link3"/>
+      <child link="cylinder2"/>
       <axis xyz="0 -1 0"/>
       <limit effort="0" lower="${radians(-90)}" upper="${0}" velocity="${radians(156)}"/>
-    </joint> -->
+    </joint>
     <joint name="tip_joint" type="fixed">
       <origin xyz="0.963823 0 -0.642519" rpy="0 0 0"/>

Commit message: Started implementation of tip velocity controller

File: crane_description/urdf/crane.xacro (robot description, xacro)
@@ -93,5 +93,5 @@
       </visual>
     </link>
-    <link name="tip"/>
+    <link name="tip_link"/>
     <joint name="joint1" type="revolute">
       <origin xyz="0 0 0.628" rpy="0 0 0"/>
@@ -146,5 +146,5 @@
       <origin xyz="0.963823 0 -0.642519" rpy="0 0 0"/>
       <parent link="link4"/>
-      <child link="tip"/>
+      <child link="tip_link"/>
     </joint>
   </xacro:macro>

Commit message: renaming

File: crane_description/urdf/crane.xacro (robot description, xacro)
@@ -101,5 +101,12 @@
       <limit effort="0" lower="${radians(-185)}" upper="${radians(185)}" velocity="${radians(156)}"/>
     </joint>
-    <joint name="actuator_joint2" type="prismatic">
+    <joint name="link2_cylinder1_joint" type="revolute">
+      <origin xyz="0.154236 0 0.156" rpy="0 0 0"/>
+      <parent link="link2"/>
+      <child link="cylinder1"/>
+      <axis xyz="0 -1 0"/>
+      <limit effort="0" lower="${radians(-90)}" upper="${0}" velocity="${radians(156)}"/>
+    </joint>
+    <joint name="cylinder1_piston1_joint" type="prismatic">
       <origin xyz="0 0 0" rpy="0 0 0"/>
       <parent link="cylinder1"/>
@@ -115,12 +122,12 @@
       <limit effort="0" lower="${radians(-90)}" upper="${0}" velocity="${radians(156)}"/>
     </joint>
-    <joint name="link2_cylinder1_joint" type="revolute">
-      <origin xyz="0.154236 0 0.156" rpy="0 0 0"/>
-      <parent link="link2"/>
-      <child link="cylinder1"/>
+    <joint name="link3_cylinder2_joint" type="revolute">
+      <origin xyz="0.767068 0 0.002395" rpy="0 0 0"/>
+      <parent link="link3"/>
+      <child link="cylinder2"/>
       <axis xyz="0 -1 0"/>
       <limit effort="0" lower="${radians(-90)}" upper="${0}" velocity="${radians(156)}"/>
     </joint>
-    <joint name="actuator_joint3" type="prismatic">
+    <joint name="cylinder2_piston2_joint" type="prismatic">
       <origin xyz="0 0 0" rpy="0 0 0"/>
       <parent link="cylinder2"/>
@@ -136,11 +143,4 @@
       <limit effort="0" lower="${radians(-90)}" upper="${0}" velocity="${radians(156)}"/>
     </joint>
-    <joint name="link3_cylinder2_joint" type="revolute">
-      <origin xyz="0.767068 0 0.002395" rpy="0 0 0"/>
-      <parent link="link3"/>
-      <child link="cylinder2"/>
-      <axis xyz="0 -1 0"/>
-      <limit effort="0" lower="${radians(-90)}" upper="${0}" velocity="${radians(156)}"/>
-    </joint>
     <joint name="tip_joint" type="fixed">
       <origin xyz="0.963823 0 -0.642519" rpy="0 0 0"/>

Commit message: Changed origin of pistons

File: crane_description/urdf/crane.xacro (robot description, xacro)
@@ -123,5 +123,5 @@
     </joint>
     <joint name="link3_cylinder2_joint" type="revolute">
-      <origin xyz="0.767068 0 0.002395" rpy="0 0 0"/>
+      <origin xyz="0.75020 0 -0.160" rpy="0 0 0"/>
       <parent link="link3"/>
       <child link="cylinder2"/>

Commit message: actuator states

File: crane_description/urdf/crane.xacro (robot description, xacro)
@@ -108,5 +108,5 @@
       <limit effort="0" lower="${radians(-90)}" upper="${0}" velocity="${radians(156)}"/>
     </joint>
-    <joint name="cylinder1_piston1_joint" type="prismatic">
+    <joint name="actuator2" type="prismatic">
       <origin xyz="0 0 0" rpy="0 0 0"/>
       <parent link="cylinder1"/>
@@ -129,5 +129,5 @@
       <limit effort="0" lower="${radians(-90)}" upper="${0}" velocity="${radians(156)}"/>
     </joint>
-    <joint name="cylinder2_piston2_joint" type="prismatic">
+    <joint name="actuator3" type="prismatic">
       <origin xyz="0 0 0" rpy="0 0 0"/>
       <parent link="cylinder2"/>

Commit message: Working visualization of crane and pendulum

File: crane_description/urdf/crane.xacro (robot description, xacro)
@@ -94,4 +94,5 @@
     </link>
     <link name="tip_link"/>
+    <link name="suspension_frame"/>
     <joint name="joint1" type="revolute">
       <origin xyz="0 0 0.628" rpy="0 0 0"/>
@@ -148,4 +149,10 @@
       <child link="tip_link"/>
     </joint>
+    <joint name="suspension_joint" type="continuous">
+      <origin xyz="0 0 0" rpy="0 0 0"/>
+      <parent link="tip_link"/>
+      <child link="suspension_frame"/>
+      <axis xyz="0 -1 0"/>
+    </joint>
   </xacro:macro>
 </robot>

File: crane_description/urdf/crane_with_pendulum.urdf.xacro (robot description, xacro)
@@ -3,11 +3,10 @@
   <xacro:include filename="$(find crane_description)/urdf/crane.xacro" />
   <xacro:include filename="$(find crane_description)/urdf/pendulum.xacro" />
-  <xacro:pendulum prefix="crane" />
-  <xacro:pendulum prefix="pendulum" length="1.05" />
-  <link name="world"/>
+  <xacro:crane />
+  <xacro:pendulum prefix="pendulum_" length="1.05" />
   <joint name="crane_tip_pendulum" type="fixed">
     <origin xyz="0 0 0" rpy="0 ${radians(180)} 0"/>
-    <parent link="world"/>
-    <child link="base_link"/>
+    <parent link="suspension_frame"/>
+    <child link="pendulum_base_link"/>
   </joint>
 </robot>

File: crane_description/urdf/pendulum.xacro (robot description, xacro)
@@ -2,14 +2,14 @@
 <robot xmlns:xacro="http://www.ros.org/wiki/xacro">
   <xacro:macro name="pendulum" params="prefix length">
-    <material name="white">
+    <material name="${prefix}white">
       <color rgba="1 1 1 1"/>
     </material>
-    <material name="gray">
+    <material name="${prefix}gray">
       <color rgba="0.5 0.5 0.5 1"/>
     </material>
-    <material name="lessgray">
+    <material name="${prefix}lessgray">
       <color rgba="0.75 0.75 0.75 1"/>
     </material>
-    <material name="red">
+    <material name="${prefix}red">
       <color rgba="1 0 0 1"/>
     </material>
@@ -37,5 +37,5 @@
           <cylinder radius="0.005" length="${length}"/>
         </geometry>
-        <material name="lessgray"/>
+        <material name="${prefix}lessgray"/>
       </visual>
     </link>
@@ -50,5 +50,5 @@
           <sphere radius="0.1"/>
         </geometry>
-        <material name="red"/>
+        <material name="${prefix}red"/>
       </visual>
     </link>

Commit message: Nearly there!

File: crane_description/urdf/crane.xacro (robot description, xacro)
@@ -94,4 +94,5 @@
     </link>
     <link name="tip_link"/>
+    <link name="suspension_frame1"/>
     <link name="suspension_frame"/>
     <joint name="joint1" type="revolute">
@@ -149,9 +150,15 @@
       <child link="tip_link"/>
     </joint>
-    <joint name="suspension_joint" type="continuous">
+    <joint name="suspension_joint1" type="continuous">
       <origin xyz="0 0 0" rpy="0 0 0"/>
       <parent link="tip_link"/>
+      <child link="suspension_frame1"/>
+      <axis xyz="0 -1 0"/>
+    </joint>
+    <joint name="suspension_joint2" type="continuous">
+      <origin xyz="0 0 0" rpy="0 0 0"/>
+      <axis xyz="0 0 1"/>
+      <parent link="suspension_frame1"/>
       <child link="suspension_frame"/>
-      <axis xyz="0 -1 0"/>
     </joint>
   </xacro:macro>

Commit message: Fixing frames

File: crane_description/urdf/crane.xacro (robot description, xacro)
@@ -12,4 +12,10 @@
     </material>
     <link name="base_link"/>
+    <joint name="base_link_command_frame_fixed" type="fixed">
+      <parent link="base_link"/>
+      <child link="command_frame"/>
+      <origin xyz="0 0 0" rpy="0 ${radians(180)} ${radians(-90)}"/>
+    </joint>
+    <link name="command_frame"/>
     <joint name="fixed" type="fixed">
       <parent link="base_link"/>

File: crane_description/urdf/crane_with_pendulum.urdf.xacro (robot description, xacro)
@@ -6,5 +6,5 @@
   <xacro:pendulum prefix="pendulum_" length="1.05" />
   <joint name="crane_tip_pendulum" type="fixed">
-    <origin xyz="0 0 0" rpy="0 ${radians(180)} 0"/>
+    <origin xyz="0 0 0" rpy="0 ${radians(180)} ${radians(-90)}"/>
     <parent link="suspension_frame"/>
     <child link="pendulum_base_link"/>
